File: Projeto 02 - Hardware Front End/frontEnd.sch (KiCad schematic (older format))
At the start: 22 parts, among them J1 Power_Supply, J2 Signal_Input, J3 MCU_Interface, U1 L78L12_TO92, U2 L79L12_TO92, U3 LM311

Commit message: Projeto CCS quase 100%
Parts:
- removed R3: 22k, Resistor_THT:R_Axial_DIN0207_L6.3mm_D2.5mm_P10.16mm_Horizontal, symbol Device:R
- R2: value 2.2k -> 68k
Connections:
- wire segments 75 -> 72
Changed lines of the file:
@@
 EESchema Schematic File Version 4
+LIBS:frontEnd-cache
 EELAYER 26 0
 EELAYER END
@@
 $EndDescr
 $Comp
-L Device:R R1
-U 1 1 5BC0B5B1
-P 2650 3900
-F 0 "R1" V 2443 3900 50  0000 C CNN
-F 1 "1k" V 2534 3900 50  0000 C CNN
-F 2 "Resistor_THT:R_Axial_DIN0207_L6.3mm_D2.5mm_P10.16mm_Horizontal" V 2580 3900 50  0001 C CNN
-F 3 "~" H 2650 3900 50  0001 C CNN
-	1    2650 3900
-	0    1    1    0
-$EndComp
-$Comp
 L Device:R R4
 U 1 1 5BC0B607
-P 4050 4200
-F 0 "R4" H 3980 4154 50  0000 R CNN
-F 1 "1M" H 3980 4245 50  0000 R CNN
-F 2 "Resistor_THT:R_Axial_DIN0207_L6.3mm_D2.5mm_P10.16mm_Horizontal" V 3980 4200 50  0001 C CNN
-F 3 "~" H 4050 4200 50  0001 C CNN
-	1    4050 4200
+P 4100 4200
+F 0 "R4" H 4030 4154 50  0000 R CNN
+F 1 "1M" H 4030 4245 50  0000 R CNN
+F 2 "Resistor_THT:R_Axial_DIN0207_L6.3mm_D2.5mm_P10.16mm_Horizontal" V 4030 4200 50  0001 C CNN
+F 3 "~" H 4100 4200 50  0001 C CNN
+	1    4100 4200
 	-1   0    0    1
 $EndComp
@@
 L Device:C C3
 U 1 1 5BC0B6B0
-P 3750 3900
-F 0 "C3" V 3498 3900 50  0000 C CNN
-F 1 "68u" V 3589 3900 50  0000 C CNN
-F 2 "Capacitor_THT:C_Rect_L29.0mm_W11.9mm_P27.50mm_MKT" H 3788 3750 50  0001 C CNN
-F 3 "~" H 3750 3900 50  0001 C CNN
-	1    3750 3900
+P 2900 3900
+F 0 "C3" V 2648 3900 50  0000 C CNN
+F 1 "68u" V 2739 3900 50  0000 C CNN
+F 2 "Capacitor_THT:C_Rect_L29.0mm_W11.9mm_P27.50mm_MKT" H 2938 3750 50  0001 C CNN
+F 3 "~" H 2900 3900 50  0001 C CNN
+	1    2900 3900
 	0    1    1    0
 $EndComp
 Wire Wire Line
-	2800 3900 2950 3900
-Wire Wire Line
-	2950 4050 2950 3900
-Connection ~ 2950 3900
-Wire Wire Line
-	2950 3750 2950 3900
-Wire Wire Line
-	4050 4050 4050 3900
+	3700 4050 3700 3900
+Connection ~ 3700 3900
+Wire Wire Line
+	3700 3750 3700 3900
+Wire Wire Line
+	4100 4050 4100 3900
 $Comp
 L Connector:Conn_01x02_Male J2
@@
 	1    0    0    -1
 $EndComp
-Wire Wire Line
-	2500 3900 2200 3900
 $Comp
 L power:GND #PWR0101
@@
 L power:GND #PWR0102
 U 1 1 5BC0BB60
-P 4050 4400
-F 0 "#PWR0102" H 4050 4150 50  0001 C CNN
-F 1 "GND" H 4055 4227 50  0000 C CNN
-F 2 "" H 4050 4400 50  0001 C CNN
-F 3 "" H 4050 4400 50  0001 C CNN
-	1    4050 4400
-	1    0    0    -1
-$EndComp
-Wire Wire Line
-	4050 4400 4050 4350
+P 4100 4400
+F 0 "#PWR0102" H 4100 4150 50  0001 C CNN
+F 1 "GND" H 4105 4227 50  0000 C CNN
+F 2 "" H 4100 4400 50  0001 C CNN
+F 3 "" H 4100 4400 50  0001 C CNN
+	1    4100 4400
+	1    0    0    -1
+$EndComp
+Wire Wire Line
+	4100 4400 4100 4350
 $Comp
 L Comparator:LM311 U3
@@
 	1    0    0    -1
 $EndComp
-Wire Wire Line
-	4050 3900 4550 3900
 $Comp
 L power:GND #PWR0103
@@
 L Device:D D1
 U 1 1 5BC0C9E3
-P 2950 3600
-F 0 "D1" V 2904 3679 50  0000 L CNN
-F 1 "D" V 2995 3679 50  0000 L CNN
-F 2 "Diode_THT:D_DO-35_SOD27_P5.08mm_Vertical_KathodeUp" H 2950 3600 50  0001 C CNN
-F 3 "~" H 2950 3600 50  0001 C CNN
-	1    2950 3600
+P 3700 3600
+F 0 "D1" V 3654 3679 50  0000 L CNN
+F 1 "D" V 3745 3679 50  0000 L CNN
+F 2 "Diode_THT:D_DO-35_SOD27_P5.08mm_Vertical_KathodeUp" H 3700 3600 50  0001 C CNN
+F 3 "~" H 3700 3600 50  0001 C CNN
+	1    3700 3600
 	0    1    1    0
 $EndComp
@@
 L Device:D D2
 U 1 1 5BC0CA31
-P 2950 4200
-F 0 "D2" V 2904 4279 50  0000 L CNN
-F 1 "D" V 2995 4279 50  0000 L CNN
-F 2 "Diode_THT:D_DO-35_SOD27_P5.08mm_Vertical_KathodeUp" H 2950 4200 50  0001 C CNN
-F 3 "~" H 2950 4200 50  0001 C CNN
-	1    2950 4200
+P 3700 4200
+F 0 "D2" V 3654 4279 50  0000 L CNN
+F 1 "D" V 3745 4279 50  0000 L CNN
+F 2 "Diode_THT:D_DO-35_SOD27_P5.08mm_Vertical_KathodeUp" H 3700 4200 50  0001 C CNN
+F 3 "~" H 3700 4200 50  0001 C CNN
+	1    3700 4200
 	0    1    1    0
 $EndComp
-Wire Wire Line
-	3900 3900 4050 3900
-Connection ~ 4050 3900
-$Comp
-L Device:R R3
-U 1 1 5BC0CC69
-P 3450 4150
-F 0 "R3" H 3380 4104 50  0000 R CNN
-F 1 "22k" H 3380 4195 50  0000 R CNN
-F 2 "Resistor_THT:R_Axial_DIN0207_L6.3mm_D2.5mm_P10.16mm_Horizontal" V 3380 4150 50  0001 C CNN
-F 3 "~" H 3450 4150 50  0001 C CNN
-	1    3450 4150
-	-1   0    0    1
-$EndComp
-$Comp
-L Device:R R2
-U 1 1 5BC0CCA5
-P 3200 3900
-F 0 "R2" V 2993 3900 50  0000 C CNN
-F 1 "2.2k" V 3084 3900 50  0000 C CNN
-F 2 "Resistor_THT:R_Axial_DIN0207_L6.3mm_D2.5mm_P10.16mm_Horizontal" V 3130 3900 50  0001 C CNN
-F 3 "~" H 3200 3900 50  0001 C CNN
-	1    3200 3900
-	0    1    1    0
-$EndComp
-Wire Wire Line
-	3050 3900 2950 3900
-Wire Wire Line
-	3350 3900 3450 3900
-Wire Wire Line
-	3450 4000 3450 3900
-Connection ~ 3450 3900
-Wire Wire Line
-	3450 3900 3600 3900
-$Comp
-L power:GND #PWR0104
-U 1 1 5BC0D350
-P 3450 4400
-F 0 "#PWR0104" H 3450 4150 50  0001 C CNN
-F 1 "GND" H 3455 4227 50  0000 C CNN
-F 2 "" H 3450 4400 50  0001 C CNN
-F 3 "" H 3450 4400 50  0001 C CNN
-	1    3450 4400
-	1    0    0    -1
-$EndComp
-Wire Wire Line
-	3450 4400 3450 4300
 $Comp
 L Connector:Conn_01x03_Male J3
@@
 L power:+12V #PWR0106
 U 1 1 5BC17F26
-P 2950 3350
-F 0 "#PWR0106" H 2950 3200 50  0001 C CNN
-F 1 "+12V" H 2965 3523 50  0000 C CNN
-F 2 "" H 2950 3350 50  0001 C CNN
-F 3 "" H 2950 3350 50  0001 C CNN
-	1    2950 3350
+P 3700 3350
+F 0 "#PWR0106" H 3700 3200 50  0001 C CNN
+F 1 "+12V" H 3715 3523 50  0000 C CNN
+F 2 "" H 3700 3350 50  0001 C CNN
+F 3 "" H 3700 3350 50  0001 C CNN
+	1    3700 3350
 	1    0    0    -1
 $EndComp
@@
 L power:-12V #PWR0107
 U 1 1 5BC17F93
-P 2950 4450
-F 0 "#PWR0107" H 2950 4550 50  0001 C CNN
-F 1 "-12V" H 2965 4623 50  0000 C CNN
-F 2 "" H 2950 4450 50  0001 C CNN
-F 3 "" H 2950 4450 50  0001 C CNN
-	1    2950 4450
+P 3700 4450
+F 0 "#PWR0107" H 3700 4550 50  0001 C CNN
+F 1 "-12V" H 3715 4623 50  0000 C CNN
+F 2 "" H 3700 4450 50  0001 C CNN
+F 3 "" H 3700 4450 50  0001 C CNN
+	1    3700 4450
 	-1   0    0    1
 $EndComp
@@
 	4750 3650 4750 3700
 Wire Wire Line
-	2950 4450 2950 4350
-Wire Wire Line
-	2950 3350 2950 3450
+	3700 4450 3700 4350
+Wire Wire Line
+	3700 3350 3700 3450
+$Comp
+L Device:R R1
+U 1 1 5BC3D5B6
+P 3300 3900
+F 0 "R1" H 3230 3854 50  0000 R CNN
+F 1 "1k" H 3230 3945 50  0000 R CNN
+F 2 "Resistor_THT:R_Axial_DIN0207_L6.3mm_D2.5mm_P10.16mm_Horizontal" V 3230 3900 50  0001 C CNN
+F 3 "~" H 3300 3900 50  0001 C CNN
+	1    3300 3900
+	0    -1   -1   0
+$EndComp
+Wire Wire Line
+	3050 3900 3150 3900
+Wire Wire Line
+	2200 3900 2750 3900
+Wire Wire Line
+	3700 3900 3450 3900
+$Comp
+L Device:R R2
+U 1 1 5BC45BDB
+P 3900 3900
+F 0 "R2" H 3830 3854 50  0000 R CNN
+F 1 "68k" H 3830 3945 50  0000 R CNN
+F 2 "Resistor_THT:R_Axial_DIN0207_L6.3mm_D2.5mm_P10.16mm_Horizontal" V 3830 3900 50  0001 C CNN
+F 3 "~" H 3900 3900 50  0001 C CNN
+	1    3900 3900
+	0    -1   -1   0
+$EndComp
+Wire Wire Line
+	3750 3900 3700 3900
+Wire Wire Line
+	4050 3900 4100 3900
+Wire Wire Line
+	4100 3900 4550 3900
+Connection ~ 4100 3900
 $EndSCHEMATC
